Commit message: New test added

File: fusion2urdf-master/Example/Basic_Robot_description/urdf/Basic_Robot.xacro (robot description, xacro)
@@ -6,10 +6,10 @@
 <link name="base_link">
   <inertial>
-    <origin xyz="0.08324805143827513 0.0009581969043022348 -0.06183590609707082" rpy="0 0 0"/>
+    <origin rpy="0 0 0" xyz="0.047517484701943946 0.004858805619815502 -0.0300059480762529"/>
     <mass value="0.4424914005445932"/>
-    <inertia ixx="0.000128" iyy="0.00046" izz="0.000341" ixy="2e-06" iyz="0.0" ixz="-0.0"/>
+    <inertia ixx="0.000128" ixy="2e-06" ixz="-0.0" iyy="0.00046" iyz="0.0" izz="0.000341"/>
   </inertial>
   <visual>
-    <origin xyz="0 0 0" rpy="0 0 0"/>
+    <origin rpy="0 0 0" xyz="0 0 0"/>
     <geometry>
       <mesh filename="package://Basic_Robot_description/meshes/base_link.stl" scale="0.001 0.001 0.001"/>
@@ -18,5 +18,5 @@
   </visual>
   <collision>
-    <origin xyz="0 0 0" rpy="0 0 0"/>
+    <origin rpy="0 0 0" xyz="0 0 0"/>
     <geometry>
       <mesh filename="package://Basic_Robot_description/meshes/base_link.stl" scale="0.001 0.001 0.001"/>
@@ -26,10 +26,10 @@
 <link name="right_wheel_1">
   <inertial>
-    <origin xyz="-0.030730433263668804 0.0039003912844867332 0.03040242803816333" rpy="0 0 0"/>
+    <origin rpy="0 0 0" xyz="0.005000000000000007 4.336808689942018e-18 -0.001427613941018771"/>
     <mass value="0.015522874373267303"/>
-    <inertia ixx="1e-06" iyy="1e-06" izz="2e-06" ixy="0.0" iyz="0.0" ixz="-0.0"/>
+    <inertia ixx="1e-06" ixy="0.0" ixz="-0.0" iyy="1e-06" iyz="0.0" izz="2e-06"/>
   </inertial>
   <visual>
-    <origin xyz="-0.071461 0.002801 0.12366" rpy="0 0 0"/>
+    <origin rpy="0 0 0" xyz="-0.0 -0.005 0.06"/>
     <geometry>
       <mesh filename="package://Basic_Robot_description/meshes/right_wheel_1.stl" scale="0.001 0.001 0.001"/>
@@ -38,5 +38,5 @@
   </visual>
   <collision>
-    <origin xyz="-0.071461 0.002801 0.12366" rpy="0 0 0"/>
+    <origin rpy="0 0 0" xyz="-0.0 -0.005 0.06"/>
     <geometry>
       <mesh filename="package://Basic_Robot_description/meshes/right_wheel_1.stl" scale="0.001 0.001 0.001"/>
@@ -46,10 +46,10 @@
 <link name="left_wheel_1">
   <inertial>
-    <origin xyz="-0.03073043326366881 0.0039003912844867324 0.03325765592020084" rpy="0 0 0"/>
+    <origin rpy="0 0 0" xyz="0.004999999999999999 0.0 0.0014276139410187671"/>
     <mass value="0.015522874373267314"/>
-    <inertia ixx="1e-06" iyy="1e-06" izz="2e-06" ixy="-0.0" iyz="0.0" ixz="-0.0"/>
+    <inertia ixx="1e-06" ixy="-0.0" ixz="-0.0" iyy="1e-06" iyz="0.0" izz="2e-06"/>
   </inertial>
   <visual>
-    <origin xyz="-0.071461 0.002801 0.06366" rpy="0 0 0"/>
+    <origin rpy="0 0 0" xyz="-0.0 -0.005 -0.0"/>
     <geometry>
       <mesh filename="package://Basic_Robot_description/meshes/left_wheel_1.stl" scale="0.001 0.001 0.001"/>
@@ -58,5 +58,5 @@
   </visual>
   <collision>
-    <origin xyz="-0.071461 0.002801 0.06366" rpy="0 0 0"/>
+    <origin rpy="0 0 0" xyz="-0.0 -0.005 -0.0"/>
     <geometry>
       <mesh filename="package://Basic_Robot_description/meshes/left_wheel_1.stl" scale="0.001 0.001 0.001"/>
@@ -64,12 +64,12 @@
   </collision>
 </link>
-<joint name="Revoluci�n1" type="continuous">
-  <origin xyz="0.071461 -0.002801 -0.12366" rpy="0 0 0"/>
+<joint name="Rev1" type="continuous">
+  <origin rpy="0 0 0" xyz="0.0 0.005 -0.06"/>
   <parent link="base_link"/>
   <child link="right_wheel_1"/>
-  <axis xyz="-0.0 -0.0 -1.0"/>
+  <axis xyz="0.0 0.0 -1.0"/>
 </joint>
-<joint name="Revoluci�n2" type="continuous">
-  <origin xyz="0.071461 -0.002801 -0.06366" rpy="0 0 0"/>
+<joint name="Rev2" type="continuous">
+  <origin rpy="0 0 0" xyz="0.0 0.005 0.0"/>
   <parent link="base_link"/>
   <child link="left_wheel_1"/>
