Commit message: Update materials.xacro

File: Spot_arm/Spot_Arm_Export_description/urdf/materials.xacro (robot description, xacro)
@@ -1,6 +1,12 @@
 <?xml version="1.0" ?>
 <robot name="Spot_Arm_Export" xmlns:xacro="http://www.ros.org/wiki/xacro" >
+<material name="yellow">
+  <color rgba="0.992 0.8705 0.08235 1.000"/>
+</material>
+<material name="black">
+  <color rgba="0.254 0.254 0.235 1.000"/>
+</material>
 <material name="silver">
-  <color rgba="0.700 0.700 0.700 1.000"/>
+  <color rgba="0.4627 0.4627 0.4549 1.000"/>
 </material>
 </robot>
