Commit message: Update Spot_Arm_Export.xacro

File: Spot_arm/Spot_Arm_Export_description/urdf/Spot_Arm_Export.xacro (robot description, xacro)
@@ -193,5 +193,5 @@
   <child link="link5_1"/>
   <axis xyz="1.0 -0.0 0.0"/>
-  <limit upper="0.0" lower="0.0" effort="100" velocity="100"/>
+  <limit upper="0.0" lower="0.05" effort="100" velocity="100"/>
 </joint>
 <joint name="Rev14" type="continuous">

Commit message: Update Spot_Arm_Export.xacro

File: Spot_arm/Spot_Arm_Export_description/urdf/Spot_Arm_Export.xacro (robot description, xacro)
@@ -164,21 +164,24 @@
   </collision>
 </link>
-<joint name="Rev7" type="continuous">
+<joint name="Rev7" type="revolute">
   <origin xyz="0.0 0.0 0.04" rpy="0 0 0"/>
   <parent link="base_link"/>
   <child link="link1_1"/>
   <axis xyz="0.0 0.0 1.0"/>
-</joint>
-<joint name="Rev8" type="continuous">
+  <limit effort="500.0" lower="-2.61799" upper="3.14159" velocity="0.5"/>
+</joint>
+<joint name="Rev8" type="revolute">
   <origin xyz="0.0 0.03 0.1" rpy="0 0 0"/>
   <parent link="link1_1"/>
   <child link="link2__1"/>
   <axis xyz="0.0 -1.0 0.0"/>
-</joint>
-<joint name="Rev9" type="continuous">
+  <limit effort="500.0" lower="-0.523599" upper="3.14159" velocity="0.5"/>
+</joint>
+<joint name="Rev9" type="revolute">
   <origin xyz="0.3385 -0.02 0.000137" rpy="0 0 0"/>
   <parent link="link2__1"/>
   <child link="link3_1"/>
   <axis xyz="0.0 1.0 0.0"/>
+  <limit effort="500.0" lower="0" upper="2.61799" velocity="0.5"/>
 </joint>
 <joint name="Rev10" type="continuous">
@@ -186,5 +189,5 @@
   <parent link="link3_1"/>
   <child link="link4_1"/>
-  <axis xyz="1.0 0.0 0.0"/>
+  <limit effort="500.0" lower="-4.3633" upper="1.22173" velocity="0.5"/>
 </joint>
 <joint name="Slider11" type="prismatic">
@@ -193,17 +196,19 @@
   <child link="link5_1"/>
   <axis xyz="1.0 -0.0 0.0"/>
-  <limit upper="0.0" lower="0.05" effort="100" velocity="100"/>
-</joint>
-<joint name="Rev14" type="continuous">
+  <limit upper="0.075" lower="0.0" effort="100" velocity="100"/>
+</joint>
+<joint name="Rev14" type="revolute">
   <origin xyz="0.2413 0.01 0.0" rpy="0 0 0"/>
   <parent link="link5_1"/>
   <child link="link6_1"/>
   <axis xyz="-0.0 1.0 0.0"/>
-</joint>
-<joint name="Rev15" type="continuous">
+  <limit effort="500.0" lower="-1.047198" upper="1.047198" velocity="0.5"/>
+</joint>
+<joint name="Rev15" type="revolute">
   <origin xyz="0.1 -0.0105 0.0" rpy="0 0 0"/>
   <parent link="link6_1"/>
   <child link="link7_1"/>
   <axis xyz="-1.0 -0.0 -0.0"/>
+  <limit effort="500.0" lower="-4.45059" upper="1.30899" velocity="0.5"/>
 </joint>
 </robot>

Commit message: Update Spot_Arm_Export.xacro

File: Spot_arm/Spot_Arm_Export_description/urdf/Spot_Arm_Export.xacro (robot description, xacro)
@@ -185,5 +185,5 @@
   <limit effort="500.0" lower="0" upper="2.61799" velocity="0.5"/>
 </joint>
-<joint name="Rev10" type="continuous">
+<joint name="Rev10" type="revolute">
   <origin xyz="0.107 -0.01 0.09734" rpy="0 0 0"/>
   <parent link="link3_1"/>

Commit message: Update Spot_Arm_Export.xacro

File: Spot_arm/Spot_Arm_Export_description/urdf/Spot_Arm_Export.xacro (robot description, xacro)
@@ -15,5 +15,5 @@
       <mesh filename="package://Spot_Arm_Export_description/meshes/base_link.stl" scale="0.001 0.001 0.001"/>
     </geometry>
-    <material name="silver"/>
+    <material name="black"/>
   </visual>
   <collision>
@@ -35,5 +35,5 @@
       <mesh filename="package://Spot_Arm_Export_description/meshes/link1_1.stl" scale="0.001 0.001 0.001"/>
     </geometry>
-    <material name="silver"/>
+    <material name="black"/>
   </visual>
   <collision>
@@ -55,5 +55,5 @@
       <mesh filename="package://Spot_Arm_Export_description/meshes/link2__1.stl" scale="0.001 0.001 0.001"/>
     </geometry>
-    <material name="silver"/>
+    <material name="yellow"/>
   </visual>
   <collision>
@@ -115,5 +115,5 @@
       <mesh filename="package://Spot_Arm_Export_description/meshes/link5_1.stl" scale="0.001 0.001 0.001"/>
     </geometry>
-    <material name="silver"/>
+    <material name="yellow"/>
   </visual>
   <collision>
@@ -155,5 +155,5 @@
       <mesh filename="package://Spot_Arm_Export_description/meshes/link7_1.stl" scale="0.001 0.001 0.001"/>
     </geometry>
-    <material name="silver"/>
+    <material name="black"/>
   </visual>
   <collision>
